File: Regulador_tensao_5v_usba_3_3v.kicad_pcb (KiCad board)
At the start: 2 copper layers, 17 parts, among them J1 USB_A, J2 Screw_Terminal_01x02, J3 Barrel_Jack, U1 LM7805_TO220, U2 LD1117V33

Commit message: Add files via upload
Other:
- board outline added: 124.8 x 71.2 mm
Changed lines of the file:
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@@
 		(layer "F.Cu")
+	)
+	(gr_rect
+		(start 83.2 89.6)
+		(end 208 160.8)
+		(stroke
+			(width 0.05)
+			(type default)
+		)
+		(fill no)
+		(layer "Edge.Cuts")
 	)
 	(segment
